File: pcb/macjis.kicad_pcb (KiCad board)
At the start: 2 copper layers, 287.8 x 136.3 mm, 178 parts, among them SW1 SW_Hotswap_Kailh_Choc_V1V2, SW10 SW_Hotswap_Kailh_Choc_V1V2, SW11 SW_Hotswap_Kailh_Choc_V1V2, SW12 SW_Hotswap_Kailh_Choc_V1V2, SW13 SW_Hotswap_Kailh_Choc_V1V2, SW14 SW_Hotswap_Kailh_Choc_V1V2, SW15 SW_Hotswap_Kailh_Choc_V1V2, SW16 SW_Hotswap_Kailh_Choc_V1V2, SW17 SW_Hotswap_Kailh_Choc_V1V2, SW18 SW_Hotswap_Kailh_Choc_V1V2, SW19 SW_Hotswap_Kailh_Choc_V1V2, SW2 SW_Hotswap_Kailh_Choc_V1V2, SW20 SW_Hotswap_Kailh_Choc_V1V2, SW21 SW_Hotswap_Kailh_Choc_V1V2, SW22 SW_Hotswap_Kailh_Choc_V1V2, SW23 SW_Hotswap_Kailh_Choc_V1V2, SW24 SW_Hotswap_Kailh_Choc_V1V2, SW25 SW_Hotswap_Kailh_Choc_V1V2, SW26 SW_Hotswap_Kailh_Choc_V1V2, SW27 SW_Hotswap_Kailh_Choc_V1V2, SW28 SW_Hotswap_Kailh_Choc_V1V2, SW29 SW_Hotswap_Kailh_Choc_V1V2, SW3 SW_Hotswap_Kailh_Choc_V1V2, SW30 SW_Hotswap_Kailh_Choc_V1V2, SW31 SW_Hotswap_Kailh_Choc_V1V2, SW32 SW_Hotswap_Kailh_Choc_V1V2, SW33 SW_Hotswap_Kailh_Choc_V1V2, SW34 SW_Hotswap_Kailh_Choc_V1V2, SW35 SW_Hotswap_Kailh_Choc_V1V2, SW36 SW_Hotswap_Kailh_Choc_V1V2, SW37 SW_Hotswap_Kailh_Choc_V1V2, SW38 SW_Hotswap_Kailh_Choc_V1V2, SW39 SW_Hotswap_Kailh_Choc_V1V2, SW4 SW_Hotswap_Kailh_Choc_V1V2, SW40 SW_Hotswap_Kailh_Choc_V1V2, SW41 SW_Hotswap_Kailh_Choc_V1V2, SW42 SW_Hotswap_Kailh_Choc_V1V2, SW43 SW_Hotswap_Kailh_Choc_V1V2, SW44 SW_Hotswap_Kailh_Choc_V1V2, SW44_2 SW_Hotswap_Kailh_Choc_V1V2, SW45 SW_Hotswap_Kailh_Choc_V1V2, SW46 SW_Hotswap_Kailh_Choc_V1V2, SW47 SW_Hotswap_Kailh_Choc_V1V2, SW48 SW_Hotswap_Kailh_Choc_V1V2, SW49 SW_Hotswap_Kailh_Choc_V1V2, SW5 SW_Hotswap_Kailh_Choc_V1V2, SW50 SW_Hotswap_Kailh_Choc_V1V2, SW51 SW_Hotswap_Kailh_Choc_V1V2, SW52 SW_Hotswap_Kailh_Choc_V1V2, SW53 SW_Hotswap_Kailh_Choc_V1V2, SW54 SW_Hotswap_Kailh_Choc_V1V2, SW55 SW_Hotswap_Kailh_Choc_V1V2, SW56 SW_Hotswap_Kailh_Choc_V1V2, SW57 SW_Hotswap_Kailh_Choc_V1V2, SW58 SW_Hotswap_Kailh_Choc_V1V2, SW58_2 SW_Hotswap_Kailh_Choc_V1V2, SW59 SW_Hotswap_Kailh_Choc_V1V2, SW6 SW_Hotswap_Kailh_Choc_V1V2, SW60 SW_Hotswap_Kailh_Choc_V1V2, SW61 SW_Hotswap_Kailh_Choc_V1V2, SW62 SW_Hotswap_Kailh_Choc_V1V2, SW63 SW_Hotswap_Kailh_Choc_V1V2, SW64 SW_Hotswap_Kailh_Choc_V1V2, SW65 SW_Hotswap_Kailh_Choc_V1V2, SW66 SW_Hotswap_Kailh_Choc_V1V2, SW67 SW_Hotswap_Kailh_Choc_V1V2, SW68 SW_Hotswap_Kailh_Choc_V1V2, SW69 SW_Hotswap_Kailh_Choc_V1V2, SW7 SW_Hotswap_Kailh_Choc_V1V2, SW70 SW_Hotswap_Kailh_Choc_V1V2, SW71 SW_Hotswap_Kailh_Choc_V1V2, SW72 SW_Hotswap_Kailh_Choc_V1V2, SW73 SW_Hotswap_Kailh_Choc_V1V2, SW74 SW_Hotswap_Kailh_Choc_V1V2, SW75 SW_Hotswap_Kailh_Choc_V1V2, SW75_2 SW_Hotswap_Kailh_Choc_V1V2, SW75_3 SW_Hotswap_Kailh_Choc_V1V2, SW76 SW_Hotswap_Kailh_Choc_V1V2, SW77 SW_Hotswap_Kailh_Choc_V1V2, SW78 SW_Hotswap_Kailh_Choc_V1V2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

Commit message: XIAO extra pads: plated holes for soldering from the back; reroute
Co-Authored-By: Claude Opus 5.5 <noreply@anthropic.com>
Claude-Session: https://claude.ai/code/session_01M64MEgyXCv4yyqteTiebrm
Routing:
- net ROW4: track 462.0 -> 415.7 mm, vias 6 -> 3
- net ROW3: track 345.9 -> 390.9 mm, vias 13 -> 10
- net COL7: track 388.0 -> 370.0 mm, vias 6 -> 5
- net COL3: track 399.5 -> 416.8 mm, vias 5 -> 3
- net COL6: track 433.5 -> 418.2 mm, vias 9 -> 7
- net COL1: track 446.4 -> 460.2 mm, vias 3 -> 5
- net ROW0: track 314.9 -> 326.7 mm, vias 12 -> 11
- net GND: track 85.3 -> 97.0 mm, vias 1 -> 2
- net ROW5: track 421.5 -> 411.6 mm, vias 7 -> 5
- net COL5: track 359.0 -> 350.6 mm, vias 5 -> 4
- net ROW6: track 212.9 -> 219.7 mm, vias 7 -> 6
- net ROW8: track 300.6 -> 294.9 mm, vias 11 -> 7
- net BAT+: track 77.1 -> 82.1 mm, vias 0 -> 1
- net COL2: track 438.6 -> 443.5 mm, vias 3 -> 5
- net ROW7: track 228.6 -> 233.3 mm, vias 8 -> 9
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
Commit message: Space cover screws evenly between the back feet; move battery connector
Co-Authored-By: Claude Opus 5.5 <noreply@anthropic.com>
Claude-Session: https://claude.ai/code/session_01M64MEgyXCv4yyqteTiebrm
Parts:
- moved H8 64.9 mm to (79.2, -10.5)
- moved H9 28.6 mm to (142.9, -10.5)
- moved J_BAT 18.0 mm to (189.8, -13.5)
- moved H10 12.3 mm to (206.6, -10.5)
Routing:
- net ROW4: track 415.7 -> 380.1 mm, vias 3 -> 15
- net BAT+: track 82.1 -> 117.1 mm, vias 1 -> 3
- net COL4: track 416.2 -> 443.7 mm, vias 4 -> 9
- net COL7: track 370.0 -> 395.1 mm, vias 5 -> 8
- net COL0: track 474.6 -> 499.3 mm, vias 4 -> 7
- net ROW3: track 390.9 -> 370.5 mm, vias 10 -> 12
- net COL5: track 350.6 -> 367.8 mm, vias 4 -> 5
- net ROW5: track 411.6 -> 396.1 mm, vias 5 -> 7
- net COL8: track 353.2 -> 339.4 mm, vias 3 -> 5
- net ROW7: track 233.3 -> 220.1 mm, vias 9 -> 7
- net COL3: track 416.8 -> 404.0 mm, vias 3 -> 6
- net ROW2: track 358.6 -> 371.1 mm, vias 11 -> 12
- net ROW8: track 294.9 -> 286.3 mm, vias 7 -> 9
- net ROW1: track 343.2 -> 334.7 mm, vias 14 -> 13
- net COL1: track 460.2 -> 452.5 mm, vias 5 -> 7
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